File: keys.kicad_sch (KiCad schematic)
At the start: 444 parts, among them J1 USB_C_Receptacle_USB2.0_16P, J2 Screen, J3 TC2030_SWD, Q1 AO3401A, Q2 2N7002, Q3 2N7002, SW1 SW_Push, SW10 SW_Push, SW11 SW_Push, SW12 SW_Push, SW13 SW_Push, SW14 SW_Push, SW15 SW_Push, SW16 SW_Push, SW17 SW_Push, SW18 SW_Push, SW19 SW_Push, SW2 SW_Push, SW20 SW_Push, SW21 SW_Push, SW22 SW_Push, SW23 SW_Push, SW24 SW_Push, SW25 SW_Push, SW26 SW_Push, SW27 SW_Push, SW28 SW_Push, SW29 SW_Push, SW3 SW_Push, SW30 SW_Push, SW31 SW_Push, SW32 SW_Push, SW33 SW_Push, SW34 SW_Push, SW35 SW_Push, SW36 SW_Push, SW37 SW_Push, SW38 SW_Push, SW39 SW_Push, SW4 SW_Push, SW40 SW_Push, SW41 SW_Push, SW42 SW_Push, SW43 SW_Push, SW44 SW_Push, SW45 SW_Push, SW46 SW_Push, SW47 SW_Push, SW48 SW_Push, SW49 SW_Push, SW5 SW_Push, SW50 SW_Push, SW51 SW_Push, SW52 SW_Push, SW53 SW_Push, SW54 SW_Push, SW55 SW_Push, SW56 SW_Push, SW57 SW_Push, SW58 SW_Push, SW59 SW_Push, SW6 SW_Push, SW60 SW_Push, SW61 SW_Push, SW62 SW_Push, SW63 SW_Push, SW64 SW_Push, SW65 SW_Push, SW66 SW_Push, SW67 SW_Push, SW68 SW_Push, SW69 SW_Push, SW7 SW_Push, SW70 SW_Push, SW71 SW_Push, SW72 SW_Push, SW73 SW_Push, SW74 SW_Push, SW75 SW_Push, SW76 SW_Push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

Commit message: .
Parts:
- removed C1: 100nF, Capacitor_SMD:C_0805_2012Metric_Pad1.18x1.45mm_HandSolder, symbol Device:C_Small
- removed D31: bsd3c051v, PCM_Diode_SMD_AKL:D_SOD-323_HandSoldering, symbol Device:D_TVS
- removed H3, H5: MountingHole, MountingHole:MountingHole_2.2mm_M2, symbol Mechanical:MountingHole
- removed L2: blm15px121sn1d, Inductor_SMD:L_0805_2012Metric_Pad1.15x1.40mm_HandSolder, symbol Device:L
- added H10, H9: MountingHole_Pad, MountingHole:MountingHole_2.2mm_M2_DIN965_Pad_TopBottom, symbol Mechanical:MountingHole_Pad
- added J4: Pogopins, Connector_PinHeader_2.54mm:PinHeader_1x02_P2.54mm_Vertical, symbol Connector_Generic:Conn_01x02
Connections:
- net GNDPWR is gone; now on net GND: J1.A1 (GND), J1.A12 (GND), J1.B1 (GND), J1.B12 (GND), R1.2, R2.2, R3.2
- net ALERT: now also U6.13 (P0.01/XL2)
- net GND: now also H10.1, H9.1, J4.1 (Pin_1)
- net VBUS: now also J4.2 (Pin_2)
- net Earth: no longer names the net of J1.S1 (SHIELD), R3.1
Other:
- note removed: "Pull-ups for i2c"
- moved on the sheet: BT1, BT2, C100, C88, C89, C90, C91, C92, C93, C94, C95, C96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

Commit message: V1.0
Parts:
- removed TP19: D-, Keyboard_Specific:TestPoint_Pad_D1.0mm, symbol Connector:TestPoint
- removed TP20: D+, Keyboard_Specific:TestPoint_Pad_D1.0mm, symbol Connector:TestPoint
- added JP2: SolderJumper_3_Open, Jumper:SolderJumper-3_P1.3mm_Open_RoundedPad1.0x1.5mm, symbol Jumper:SolderJumper_3_Open
- BT1, BT2: footprint Connector_JST:JST_EH_B2B-EH-A_1x02_P2.50mm_Vertical -> Connector_PinHeader_2.54mm:PinHeader_1x02_P2.54mm_Vertical; now left out of the parts list
- C10, C100, C11, C12, C13, C14, C15, C16, C17, C18, C19, C20, C21, C22, C23, C24, C25, C26, C27, C28, C29, C3, C30, C31, C32, C33, C34, C35, C36, C37, C38, C39, C4, C40, C41, C42, C43, C44, C45, C46, C47, C48, C49, C5, C50, C51, C52, C53, C54, C55, C56, C57, C58, C59, C6, C60, C61, C62, C63, C64, C65, C66, C67, C68, C69, C7, C70, C71, C72, C73, C74, C75, C76, C77, C78, C79, C8, C80, C81, C82, C83, C84, C85, C86, C87, C9, C99: LCSC (none) -> C1525
- C88, C89, C91, C94, C96, C97: LCSC C23733 -> (none)
- C90, C92, C95: LCSC C52923 -> (none)
- C93: LCSC C307331 -> C1525
- C98: value 4u7 -> 4.7uF; LCSC C23733 -> (none)
- F1: value 3A -> 1A; footprint Fuse:Fuse_1206_3216Metric_Pad1.42x1.75mm_HandSolder -> Fuse:Fuse_0603_1608Metric_Pad1.05x0.95mm_HandSolder
- F2: value 2A -> 1A
- J4: now fitted
- L1: value ~ -> BLM15PX121SN1D; footprint Inductor_SMD:L_0805_2012Metric_Pad1.15x1.40mm_HandSolder -> Inductor_SMD:L_0402_1005Metric
- L3: value L_Small -> 10uH
- R1, R2, R3: footprint Resistor_SMD:R_0805_2012Metric_Pad1.20x1.40mm_HandSolder -> Keyboard_Specific:R_0402_1005Metric_Pad0.72x0.64mm_HandSolder
- R4, R5, R6: LCSC C25744 -> (none)
- R7: LCSC C25792 -> (none)
- R8: LCSC C25867 -> (none)
- R9: LCSC C25879 -> (none)
- U2: LCSC C2682616 -> (none)
- U3: LCSC C15464 -> (none)
- U6: LCSC C356849 -> (none)
Connections:
- net +5V: now also L1.2; no longer F1.2
- net GND: now also JP2.3 (B)
- net SYSOFF: now also JP2.1 (A); no longer U3.15 (SYSOFF)
- net VBUS: now also F1.1; no longer L1.1
- new net: F1.2, L1.1
- new net: JP2.2 (C), U3.15 (SYSOFF)
Other:
- moved on the sheet: L1
