File: keys.kicad_sch (KiCad schematic)
At the start: 441 parts, among them J1 USB_C_Receptacle_USB2.0_16P, J2 Screen, J3 TC2030_SWD, J4 Pogopins, Q1 AO3401A, Q2 2N7002, Q3 2N7002, SW1 SW_Push, SW10 SW_Push, SW11 SW_Push, SW12 SW_Push, SW13 SW_Push, SW14 SW_Push, SW15 SW_Push, SW16 SW_Push, SW17 SW_Push, SW18 SW_Push, SW19 SW_Push, SW2 SW_Push, SW20 SW_Push, SW21 SW_Push, SW22 SW_Push, SW23 SW_Push, SW24 SW_Push, SW25 SW_Push, SW26 SW_Push, SW27 SW_Push, SW28 SW_Push, SW29 SW_Push, SW3 SW_Push, SW30 SW_Push, SW31 SW_Push, SW32 SW_Push, SW33 SW_Push, SW34 SW_Push, SW35 SW_Push, SW36 SW_Push, SW37 SW_Push, SW38 SW_Push, SW39 SW_Push, SW4 SW_Push, SW40 SW_Push, SW41 SW_Push, SW42 SW_Push, SW43 SW_Push, SW44 SW_Push, SW45 SW_Push, SW46 SW_Push, SW47 SW_Push, SW48 SW_Push, SW49 SW_Push, SW5 SW_Push, SW50 SW_Push, SW51 SW_Push, SW52 SW_Push, SW53 SW_Push, SW54 SW_Push, SW55 SW_Push, SW56 SW_Push, SW57 SW_Push, SW58 SW_Push, SW59 SW_Push, SW6 SW_Push, SW60 SW_Push, SW61 SW_Push, SW62 SW_Push, SW63 SW_Push, SW64 SW_Push, SW65 SW_Push, SW66 SW_Push, SW67 SW_Push, SW68 SW_Push, SW69 SW_Push, SW7 SW_Push, SW70 SW_Push, SW71 SW_Push, SW72 SW_Push, SW73 SW_Push, SW74 SW_Push, SW75 SW_Push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

Commit message: Usb Connector Daugherboard ''fertig''
Parts:
- removed R3: 1M, Keyboard_Specific:R_0402_1005Metric_Pad0.72x0.64mm_HandSolder, symbol Device:R_Small
- added C1: 0.1uF, Capacitor_SMD:C_0603_1608Metric_Pad1.08x0.95mm_HandSolder, symbol Device:C_Small
- added C101: 0.001uF, Capacitor_SMD:C_0603_1608Metric_Pad1.08x0.95mm_HandSolder, symbol Device:C_Small
- added C102: 10uF, Capacitor_SMD:C_0603_1608Metric_Pad1.08x0.95mm_HandSolder, symbol Device:C_Small
- added C103, C104, C2: 0.01uF, Capacitor_SMD:C_0603_1608Metric_Pad1.08x0.95mm_HandSolder, symbol Device:C_Small
- added H11, H3, H5: MountingHole, MountingHole:MountingHole_3.2mm_M3_DIN965, symbol Mechanical:MountingHole
- added H12: MountingHole_Pad, MountingHole:MountingHole_3.2mm_M3_DIN965_Pad_TopBottom, symbol Mechanical:MountingHole_Pad
- added J5, J6: Conn_01x06_Socket, Connector_FFC-FPC:Molex_200528-0060_1x06-1MP_P1.00mm_Horizontal, symbol Connector:Conn_01x06_Socket
- added L2: BLM15PX121SN1D, Inductor_SMD:L_0402_1005Metric, symbol Device:L
- C10, C100, C11, C12, C13, C14, C15, C16, C17, C18, C19, C20, C21, C22, C23, C24, C25, C26, C27, C28, C29, C3, C30, C31, C32, C33, C34, C35, C36, C37, C38, C39, C4, C40, C41, C42, C43, C44, C45, C46, C47, C48, C49, C5, C50, C51, C52, C53, C54, C55, C56, C57, C58, C59, C6, C60, C61, C62, C63, C64, C65, C66, C67, C68, C69, C7, C70, C71, C72, C73, C74, C75, C76, C77, C78, C79, C8, C80, C81, C82, C83, C84, C85, C86, C87, C88, C89, C9, C90, C91, C92, C93, C94, C95, C96, C97, C98, C99: footprint Keyboard_Specific:C_0402_1005Metric_Pad0.74x0.62mm_HandSolder -> Capacitor_SMD:C_0603_1608Metric_Pad1.08x0.95mm_HandSolder
- H1, H2, H4, H6, H7, H8: footprint MountingHole:MountingHole_2.2mm_M2 -> MountingHole:MountingHole_3.2mm_M3_DIN965
- H10, H9: footprint MountingHole:MountingHole_2.2mm_M2_DIN965_Pad_TopBottom -> MountingHole:MountingHole_3.2mm_M3_DIN965_Pad_TopBottom
- R1, R11, R12, R13, R14, R16, R17, R18, R19, R2, R20, R6, R7, R8, R9: footprint Keyboard_Specific:R_0402_1005Metric_Pad0.72x0.64mm_HandSolder -> Resistor_SMD:R_0603_1608Metric_Pad0.98x0.95mm_HandSolder
- TP1, TP10, TP11, TP12, TP13, TP14, TP15, TP16, TP17, TP18, TP2, TP21, TP22, TP23, TP24, TP25, TP26, TP27, TP28, TP29, TP3, TP30, TP31, TP32, TP4, TP5, TP6, TP7, TP8, TP9: footprint Keyboard_Specific:TestPoint_Pad_D1.0mm -> Keyboard_Specific:TestPoint_Pad_D1.5mm
Connections:
- net +5V: now also C1.2, C101.2, C102.2, C104.1, C2.2, J5.3 (Pin_3), J5.4 (Pin_4), J6.3 (Pin_3), J6.4 (Pin_4)
- net GND: now also C1.1, C101.1, C102.1, C103.2, C104.2, C2.1, H12.1, J5.1 (Pin_1), J5.2 (Pin_2), J6.1 (Pin_1), J6.2 (Pin_2); no longer J1.A1 (GND), J1.A12 (GND), J1.B1 (GND), J1.B12 (GND)
- net USB_D+: now also U5.1 (IO1), U5.4 (IO3), J5.6 (Pin_6), J6.6 (Pin_6); no longer U5.6 (IO4)
- net USB_D-: now also U5.3 (IO2), U5.6 (IO4), J5.5 (Pin_5), J6.5 (Pin_5); no longer U5.1 (IO1)
- net at J1.S1 (SHIELD): now also L2.1
- new net: C103.1, J1.A1 (GND), J1.A12 (GND), J1.B1 (GND), J1.B12 (GND), L2.2
- no-connect marks 7 -> 5
Other:
- moved on the sheet: TP1

Commit message: v2
Parts:
- removed J5, J6: Conn_01x06_Socket, Connector_FFC-FPC:Molex_200528-0060_1x06-1MP_P1.00mm_Horizontal, symbol Connector:Conn_01x06_Socket
- added J10, J11, J14, J7: Conn_01x04, Connector_PinSocket_1.27mm:PinSocket_1x04_P1.27mm_Vertical, symbol Connector_Generic:Conn_01x04
- added J12, J13, J8, J9: Conn_01x02, Connector_PinSocket_1.27mm:PinSocket_1x02_P1.27mm_Vertical, symbol Connector_Generic:Conn_01x02
- added J5, J6: Conn_01x06_MountingPin, Connector_FFC-FPC:Molex_200528-0060_1x06-1MP_P1.00mm_Horizontal, symbol Connector_Generic_MountingPin:Conn_01x06_MountingPin
- BT1, BT2: footprint Connector_PinHeader_2.54mm:PinHeader_1x02_P2.54mm_Vertical -> Resistor_SMD:R_1206_3216Metric_Pad1.30x1.75mm_HandSolder; now not fitted
Connections:
- net +5V: now also J4.2 (Pin_2), J10.1 (Pin_1), J11.1 (Pin_1), J5.3 (Pin_3), J5.4 (Pin_4), J6.3 (Pin_3), J6.4 (Pin_4)
- net +BATT: now also J10.4 (Pin_4), J11.4 (Pin_4)
- net +VSW: now also J12.2 (Pin_2), J9.2 (Pin_2)
- net ALERT: now also J14.1 (Pin_1), J7.1 (Pin_1)
- net GND: now also J12.1 (Pin_1), J13.1 (Pin_1), J13.2 (Pin_2), J14.2 (Pin_2), J5.1 (Pin_1), J5.2 (Pin_2), J5.MP (MountPin), J6.1 (Pin_1), J6.2 (Pin_2), J6.MP (MountPin), J7.2 (Pin_2), J8.1 (Pin_1), J8.2 (Pin_2), J9.1 (Pin_1)
- net SCL: now also J14.3 (Pin_3), J7.3 (Pin_3)
- net SDA: now also J14.4 (Pin_4), J7.4 (Pin_4)
- net SYSOFF: now also J10.2 (Pin_2), J11.2 (Pin_2)
- net USB_D+: now also J5.6 (Pin_6), J6.6 (Pin_6)
- net USB_D-: now also J5.5 (Pin_5), J6.5 (Pin_5)
- net VBUS: no longer J4.2 (Pin_2)
- net ~{CHG}: now also J10.3 (Pin_3), J11.3 (Pin_3)
- net FREE: now reaches U6.42 (P1.06)
